File: hw/picocart64_v2/psram.kicad_sch (KiCad schematic)
At the start: 32 parts, among them U1 APS6404L-3SQR, U10 W25Q128JVS, U11 74LVC1G125GW, U2 APS6404L-3SQR, U3 APS6404L-3SQR, U4 APS6404L-3SQR, U5 APS6404L-3SQR, U6 APS6404L-3SQR, U7 APS6404L-3SQR, U8 APS6404L-3SQR, U9 SN74LVC138AQDRQ1

Commit message: Updated schematic to include a chin for the USB port and slightly increased the length of the SD Card chin. This should help it be more accessible once inside a shell. Updated schematic to include part numbers for all the components.
Parts:
- C1, C2, C3, C4, C5, C6, C7, C8, C9: LCSC (none) -> C1525
- C39, C40, C41, C42, C43, C44, C45, C46, C47: LCSC (none) -> C14445
- R1, R2, R62: LCSC (none) -> C406733
- U1, U2, U3, U4, U5, U6, U7, U8: LCSC (none) -> Mouser: APS6404L-3SQR-SN
- U10: LCSC (none) -> C97521
- U11: LCSC (none) -> C12519
- U9: LCSC (none) -> C7816
Changed lines of the file:
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@@
+      (effects (font (size 1.27 1.27)) hide)
+    )
+    (property "LCSC" "C1525" (id 4) (at 179.705 132.08 0)
       (effects (font (size 1.27 1.27)) hide)
     )
@@
     )
     (property "Datasheet" "~" (id 3) (at 91.44 172.72 0)
+      (effects (font (size 1.27 1.27)) hide)
+    )
+    (property "LCSC" "C14445" (id 4) (at 91.44 172.72 0)
       (effects (font (size 1.27 1.27)) hide)
     )
@@
     )
     (property "Datasheet" "https://www.ti.com/lit/ds/symlink/sn74lvc138a-q1.pdf?ts=1658089127975" (id 3) (at 190.5 45.72 0)
+      (effects (font (size 1.27 1.27)) hide)
+    )
+    (property "LCSC" "C7816" (id 4) (at 190.5 45.72 0)
       (effects (font (size 1.27 1.27)) hide)
     )
@@
       (effects (font (size 1.27 1.27)) hide)
     )
+    (property "LCSC" "C1525" (id 4) (at 95.25 81.28 0)
+      (effects (font (size 1.27 1.27)) hide)
+    )
     (pin "1")
     (pin "2")
@@
     )
     (property "Datasheet" "https://www.apmemory.com/wp-content/uploads/APS6404L-3SQR.pdf" (id 3) (at 49.53 161.29 0)
+      (effects (font (size 1.27 1.27)) hide)
+    )
+    (property "LCSC" "Mouser: APS6404L-3SQR-SN" (id 4) (at 59.69 173.99 0)
       (effects (font (size 1.27 1.27)) hide)
     )
@@
       (effects (font (size 1.27 1.27)) hide)
     )
+    (property "LCSC" "C97521" (id 4) (at 207.645 133.35 0)
+      (effects (font (size 1.27 1.27)) hide)
+    )
     (pin "1")
     (pin "2")
@@
       (effects (font (size 1.27 1.27)) hide)
     )
+    (property "LCSC" "Mouser: APS6404L-3SQR-SN" (id 4) (at 59.69 82.55 0)
+      (effects (font (size 1.27 1.27)) hide)
+    )
     (pin "1")
     (pin "2")
@@
       (effects (font (size 1.27 1.27)) hide)
     )
+    (property "LCSC" "C12519" (id 4) (at 259.08 101.6 0)
+      (effects (font (size 1.27 1.27)) hide)
+    )
     (pin "1")
     (pin "2")
@@
       (effects (font (size 1.27 1.27)) hide)
     )
+    (property "LCSC" "C1525" (id 4) (at 46.99 172.72 0)
+      (effects (font (size 1.27 1.27)) hide)
+    )
     (pin "1")
     (pin "2")
@@
       (effects (font (size 1.27 1.27)) hide)
     )
+    (property "LCSC" "C14445" (id 4) (at 43.18 34.29 0)
+      (effects (font (size 1.27 1.27)) hide)
+    )
     (pin "1")
     (pin "2")
@@
       (effects (font (size 1.27 1.27)) hide)
     )
+    (property "LCSC" "C406733" (id 4) (at 157.48 53.34 0)
+      (effects (font (size 1.27 1.27)) hide)
+    )
     (pin "1")
     (pin "2")
@@
     )
     (property "Datasheet" "https://www.apmemory.com/wp-content/uploads/APS6404L-3SQR.pdf" (id 3) (at 97.79 161.29 0)
+      (effects (font (size 1.27 1.27)) hide)
+    )
+    (property "LCSC" "Mouser: APS6404L-3SQR-SN" (id 4) (at 107.95 173.99 0)
       (effects (font (size 1.27 1.27)) hide)
     )
@@
       (effects (font (size 1.27 1.27)) hide)
     )
+    (property "LCSC" "C406733" (id 4) (at 185.293 152.527 0)
+      (effects (font (size 1.27 1.27)) hide)
+    )
     (pin "1")
     (pin "2")
@@
       (effects (font (size 1.27 1.27)) hide)
     )
+    (property "LCSC" "C1525" (id 4) (at 95.25 172.72 0)
+      (effects (font (size 1.27 1.27)) hide)
+    )
     (pin "1")
     (pin "2")
@@
     )
     (property "Datasheet" "https://www.apmemory.com/wp-content/uploads/APS6404L-3SQR.pdf" (id 3) (at 97.79 115.57 0)
+      (effects (font (size 1.27 1.27)) hide)
+    )
+    (property "LCSC" "Mouser: APS6404L-3SQR-SN" (id 4) (at 107.95 128.27 0)
       (effects (font (size 1.27 1.27)) hide)
     )
@@
       (effects (font (size 1.27 1.27)) hide)
     )
+    (property "LCSC" "Mouser: APS6404L-3SQR-SN" (id 4) (at 59.69 35.56 0)
+      (effects (font (size 1.27 1.27)) hide)
+    )
     (pin "1")
     (pin "2")
@@
       (effects (font (size 1.27 1.27)) hide)
     )
+    (property "LCSC" "C406733" (id 4) (at 166.37 46.99 0)
+      (effects (font (size 1.27 1.27)) hide)
+    )
     (pin "1")
     (pin "2")
@@
       (effects (font (size 1.27 1.27)) hide)
     )
+    (property "LCSC" "C1525" (id 4) (at 46.99 34.29 0)
+      (effects (font (size 1.27 1.27)) hide)
+    )
     (pin "1")
     (pin "2")
@@
       (effects (font (size 1.27 1.27)) hide)
     )
+    (property "LCSC" "C14445" (id 4) (at 43.18 172.72 0)
+      (effects (font (size 1.27 1.27)) hide)
+    )
     (pin "1")
     (pin "2")
@@
       (effects (font (size 1.27 1.27)) hide)
     )
+    (property "LCSC" "C14445" (id 4) (at 91.44 81.28 0)
+      (effects (font (size 1.27 1.27)) hide)
+    )
     (pin "1")
     (pin "2")
@@
     )
     (property "Datasheet" "~" (id 3) (at 91.44 127 0)
+      (effects (font (size 1.27 1.27)) hide)
+    )
+    (property "LCSC" "C14445" (id 4) (at 91.44 127 0)
       (effects (font (size 1.27 1.27)) hide)
     )
@@
     )
     (property "Datasheet" "https://www.apmemory.com/wp-content/uploads/APS6404L-3SQR.pdf" (id 3) (at 97.79 69.85 0)
+      (effects (font (size 1.27 1.27)) hide)
+    )
+    (property "LCSC" "Mouser: APS6404L-3SQR-SN" (id 4) (at 107.95 82.55 0)
       (effects (font (size 1.27 1.27)) hide)
     )
@@
       (effects (font (size 1.27 1.27)) hide)
     )
+    (property "LCSC" "C1525" (id 4) (at 46.99 81.28 0)
+      (effects (font (size 1.27 1.27)) hide)
+    )
     (pin "1")
     (pin "2")
@@
     )
     (property "Datasheet" "https://www.apmemory.com/wp-content/uploads/APS6404L-3SQR.pdf" (id 3) (at 49.53 115.57 0)
+      (effects (font (size 1.27 1.27)) hide)
+    )
+    (property "LCSC" "Mouser: APS6404L-3SQR-SN" (id 4) (at 59.69 128.27 0)
       (effects (font (size 1.27 1.27)) hide)
     )
@@
       (effects (font (size 1.27 1.27)) hide)
     )
+    (property "LCSC" "C14445" (id 4) (at 91.44 34.29 0)
+      (effects (font (size 1.27 1.27)) hide)
+    )
     (pin "1")
     (pin "2")
@@
     )
     (property "Datasheet" "https://www.apmemory.com/wp-content/uploads/APS6404L-3SQR.pdf" (id 3) (at 97.79 22.86 0)
+      (effects (font (size 1.27 1.27)) hide)
+    )
+    (property "LCSC" "Mouser: APS6404L-3SQR-SN" (id 4) (at 107.95 35.56 0)
       (effects (font (size 1.27 1.27)) hide)
     )
@@
       (effects (font (size 1.27 1.27)) hide)
     )
+    (property "LCSC" "C1525" (id 4) (at 95.25 34.29 0)
+      (effects (font (size 1.27 1.27)) hide)
+    )
     (pin "1")
     (pin "2")
@@
       (effects (font (size 1.27 1.27)) hide)
     )
+    (property "LCSC" "C1525" (id 4) (at 95.25 127 0)
+      (effects (font (size 1.27 1.27)) hide)
+    )
     (pin "1")
     (pin "2")
@@
       (effects (font (size 1.27 1.27)) hide)
     )
+    (property "LCSC" "C14445" (id 4) (at 43.18 81.28 0)
+      (effects (font (size 1.27 1.27)) hide)
+    )
     (pin "1")
     (pin "2")
@@
       (effects (font (size 1.27 1.27)) hide)
     )
+    (property "LCSC" "C14445" (id 4) (at 43.18 127 0)
+      (effects (font (size 1.27 1.27)) hide)
+    )
     (pin "1")
     (pin "2")
@@
       (effects (font (size 1.27 1.27)) hide)
     )
+    (property "LCSC" "C14445" (id 4) (at 175.895 132.08 0)
+      (effects (font (size 1.27 1.27)) hide)
+    )
     (pin "1")
     (pin "2")
@@
       (effects (font (size 1.27 1.27)) hide)
     )
+    (property "LCSC" "C1525" (id 4) (at 46.99 127 0)
+      (effects (font (size 1.27 1.27)) hide)
+    )
